File: RP2040_Fan_Controller/RP2040_Fan_Controller.kicad_pcb (KiCad board)
At the start: 2 copper layers, 68.5 x 70 mm, 30 parts

Commit message: PCB-Rev 0.3.0
Parts:
- removed R10: 10K, Resistor_THT:R_Axial_DIN0204_L3.6mm_D1.6mm_P5.08mm_Horizontal
- removed R11, R12, R13, R14, R15: 10k, Resistor_THT:R_Axial_DIN0204_L3.6mm_D1.6mm_P5.08mm_Horizontal
- added ?: , , F.Cu at (181.7, 69.8)
- added ?: , , F.Cu at (179.5, 69.8)
- added ?: , , F.Cu at (180.5, 73.2)
- added G***: LOGO, Library:LOGO, F.Cu at (162.0, 115.1)
- added J1: USB, Connector_PinHeader_2.54mm:PinHeader_1x05_P2.54mm_Horizontal, F.Cu at (197.6, 69.8)
- A1: footprint Module:RaspberryPi_Pico_Common_Unspecified -> Module:RaspberryPi_Pico_Common_THT
- R1: renamed from R4; footprint Resistor_THT:R_Axial_DIN0204_L3.6mm_D1.6mm_P5.08mm_Horizontal -> Resistor_THT:R_Axial_DIN0207_L6.3mm_D2.5mm_P7.62mm_Horizontal
- R2: renamed from R5; footprint Resistor_THT:R_Axial_DIN0204_L3.6mm_D1.6mm_P5.08mm_Horizontal -> Resistor_THT:R_Axial_DIN0207_L6.3mm_D2.5mm_P7.62mm_Horizontal
- R3: renamed from R6; footprint Resistor_THT:R_Axial_DIN0204_L3.6mm_D1.6mm_P5.08mm_Horizontal -> Resistor_THT:R_Axial_DIN0207_L6.3mm_D2.5mm_P7.62mm_Horizontal
- R4: renamed from R7; footprint Resistor_THT:R_Axial_DIN0204_L3.6mm_D1.6mm_P5.08mm_Horizontal -> Resistor_THT:R_Axial_DIN0207_L6.3mm_D2.5mm_P7.62mm_Horizontal
- R5: renamed from R8; footprint Resistor_THT:R_Axial_DIN0204_L3.6mm_D1.6mm_P5.08mm_Horizontal -> Resistor_THT:R_Axial_DIN0207_L6.3mm_D2.5mm_P7.62mm_Horizontal
- R6: renamed from R9; footprint Resistor_THT:R_Axial_DIN0204_L3.6mm_D1.6mm_P5.08mm_Horizontal -> Resistor_THT:R_Axial_DIN0207_L6.3mm_D2.5mm_P7.62mm_Horizontal
- R7: renamed from R1; footprint Resistor_THT:R_Axial_DIN0204_L3.6mm_D1.6mm_P5.08mm_Horizontal -> Resistor_THT:R_Axial_DIN0207_L6.3mm_D2.5mm_P7.62mm_Horizontal
- R8: renamed from R2; footprint Resistor_THT:R_Axial_DIN0204_L3.6mm_D1.6mm_P5.08mm_Horizontal -> Resistor_THT:R_Axial_DIN0207_L6.3mm_D2.5mm_P7.62mm_Horizontal
- R9: renamed from R3; footprint Resistor_THT:R_Axial_DIN0204_L3.6mm_D1.6mm_P5.08mm_Horizontal -> Resistor_THT:R_Axial_DIN0207_L6.3mm_D2.5mm_P7.62mm_Horizontal
- moved REF** 73.5 mm to (154.8, 125.2)
- moved REF** 59.4 mm to (154.8, 54.8)
- moved Fan6 51.8 mm to (185.6, 125.6), turned to -90 degrees
- moved TH1 46.4 mm to (197.5, 101.7), turned to 0 degrees
- moved Fan5 44.9 mm to (174.0, 125.6), turned to -90 degrees
- moved TH2 41.3 mm to (197.5, 95.2), turned to 0 degrees
- moved TH3 37.8 mm to (197.5, 88.7), turned to 0 degrees
- moved R7 32.6 mm to (200.2, 117.7), turned to 90 degrees
- moved REF** 28.5 mm to (183.6, 61.0), turned to 180 degrees
- moved R8 28.2 mm to (197.0, 117.7), turned to 90 degrees
- moved Fan1 27.8 mm to (154.5, 77.3)
- moved Fan2 27.6 mm to (154.5, 88.6)
- moved Fan3 27.4 mm to (154.5, 99.9)
- moved Fan4 27.2 mm to (154.5, 111.1)
- moved R9 24.1 mm to (193.8, 117.7), turned to 90 degrees
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Connections:
- net Net-(A1-ADC_VREF) renamed ADC_VREF
- net Net-(A1-AGND) renamed ADC_GND
- net Net-(A1-GPIO0) renamed PWM_FAN1
- net Net-(A1-GPIO11) renamed RPM_FAN6
- net Net-(A1-GPIO26_ADC0) renamed ADC_0
- net Net-(A1-GPIO27_ADC1) renamed ADC_1
- net Net-(A1-GPIO28_ADC2) renamed ADC_2
- A1 pad 10: Net-(A1-GPIO7) -> RPM_FAN4
- A1 pad 11: Net-(A1-GPIO8) -> PWM_FAN5
- A1 pad 12: Net-(A1-GPIO9) -> RPM_FAN5
- A1 pad 14: Net-(A1-GPIO10) -> PWM_FAN6
- A1 pad 2: Net-(A1-GPIO1) -> RPM_FAN1
- A1 pad 4: Net-(A1-GPIO2) -> PWM_FAN2
- A1 pad 40: unconnected-(A1-VBUS-Pad40) -> VBUS
- A1 pad 5: Net-(A1-GPIO3) -> RPM_FAN2
- A1 pad 6: Net-(A1-GPIO4) -> PWM_FAN3
- A1 pad 7: Net-(A1-GPIO5) -> RPM_FAN3
- A1 pad 9: Net-(A1-GPIO6) -> PWM_FAN4
- Fan2 pad 4: Net-(A1-GPIO1) -> PWM_FAN2
- Fan3 pad 4: Net-(A1-GPIO2) -> PWM_FAN3
- Fan4 pad 4: Net-(A1-GPIO3) -> PWM_FAN4
- Fan5 pad 4: Net-(A1-GPIO4) -> PWM_FAN5
- Fan6 pad 4: Net-(A1-GPIO5) -> PWM_FAN6
- R1 pad 2: Net-(A1-GPIO6) -> RPM_FAN1
- R2 pad 2: Net-(A1-GPIO7) -> RPM_FAN2
- R3 pad 2: Net-(A1-GPIO8) -> RPM_FAN3
- R4 pad 2: Net-(A1-GPIO9) -> RPM_FAN4
- R5 pad 2: Net-(A1-GPIO10) -> RPM_FAN5
Routing:
- net ADC_VREF: track 102.4 -> 30.3 mm
- net Net-(A1-GPIO5): track 58.1 -> 0.00 mm
- net PWM_FAN6: track 0.00 -> 50.9 mm
- net Net-(A1-GPIO4): track 49.7 -> 0.00 mm
- net PWM_FAN5: track 0.00 -> 49.0 mm
- net ADC_2: track 77.1 -> 35.8 mm
- net Net-(A1-GPIO3): track 41.3 -> 0.00 mm
- net ADC_1: track 72.6 -> 32.2 mm
- net ADC_0: track 69.3 -> 30.6 mm
- net Net-(A1-GPIO2): track 34.2 -> 0.00 mm
- net Net-(A1-GPIO1): track 29.1 -> 0.00 mm
- net PWM_FAN4: track 0.00 -> 29.0 mm
- net PWM_FAN3: track 0.00 -> 25.5 mm
- net Net-(Fan1-Tacho): track 29.8 -> 5.70 mm
- net USB_DP: track 0.00 -> 20.2 mm
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Other:
- board size 68.5 x 70 mm -> 52 x 80 mm
- board text added: "Rev: 1.0.0 MIT License Nils Stein 2025"
- board text removed: "MIT License Nils Stein 2025"
- board text removed: "Rev: 0.1.0"

Commit message: PCB-Rev 0.4.0
Parts:
- moved G*** 2.68 mm to (164.2, 113.6)
- moved R7 0.40 mm to (199.8, 117.7)
- moved ? 0.38 mm to (180.6, 72.9)
- moved R8 0.25 mm to (196.8, 117.7)
- moved ? 0.19 mm to (179.6, 69.6)
- moved ? 0.17 mm to (181.6, 69.6)
- moved R9 0.10 mm to (193.8, 117.7)
Routing:
- net ADC_GND: track 45.8 -> 0.00 mm
- net ADC_VREF: track 30.3 -> 0.00 mm
- net USB_DM: track 17.1 -> 20.1 mm
- net ADC_0: track 30.6 -> 27.9 mm
- added copper zone on B.Cu, net ADC_GND
- added copper zone on F.Cu, net ADC_VREF
Other:
- outline, holes or cut-outs redrawn
- board text added: "D+"
- board text added: "D-"
- board text added: "GND"
- board text added: "S"
- board text added: "⊕"
- board text added: "⊖"

Commit message: PCB-Rev 1.0.0
Parts:
- added G***: Toast_Invert, Library:Toast_Invert, F.Cu at (73.8, 59.2)
- R1, R2, R3, R4, R5, R6, R7, R8, R9: footprint Resistor_THT:R_Axial_DIN0207_L6.3mm_D2.5mm_P7.62mm_Horizontal -> Resistor_THT:R_Axial_DIN0204_L3.6mm_D1.6mm_P7.62mm_Horizontal
- REF** (x3): value MountingHole_4.3mm_M4 -> MountingHole_3.2mm_M3_DIN965_Pad; footprint MountingHole:MountingHole_4.3mm_M4 -> MountingHole:MountingHole_3.2mm_M3_DIN965_Pad
- REF**: value MountingHole_4.3mm_M4 -> (none); footprint MountingHole:MountingHole_4.3mm_M4 -> MountingHole:MountingHole_3.2mm_M3_DIN965_Pad
- moved Fan1 100.4 mm to (55.7, 59.8), turned to 0 degrees
- moved Fan2 100.3 mm to (55.7, 71.4), turned to 0 degrees
- moved Fan3 100.2 mm to (55.7, 83.1), turned to 0 degrees
- moved Fan4 100.2 mm to (55.7, 94.7), turned to 0 degrees
- moved Fan5 97.6 mm to (76.4, 124.3), turned to 90 degrees
- moved Fan6 97.6 mm to (88.0, 124.3), turned to 90 degrees
- moved TH3 90.9 mm to (107.5, 75.7)
- moved TH2 90.7 mm to (107.5, 83.8)
- moved J1 90.6 mm to (107.5, 59.8)
- moved R2 90.6 mm to (70.0, 72.5)
- moved R7 90.6 mm to (109.8, 107.7)
- moved R8 90.6 mm to (106.8, 107.7)
- moved R9 90.6 mm to (103.8, 107.7)
- moved REF** 90.6 mm to (64.8, 44.8)
- moved REF** 90.6 mm to (93.6, 51.0)
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Connections:
- A1 pad 1: PWM_FAN1 -> unconnected-(A1-GPIO0-Pad1)
- A1 pad 10: RPM_FAN4 -> PWM_FAN3
- A1 pad 11: PWM_FAN5 -> RPM_FAN4
- A1 pad 12: RPM_FAN5 -> PWM_FAN4
- A1 pad 14: PWM_FAN6 -> RPM_FAN5
- A1 pad 15: RPM_FAN6 -> PWM_FAN5
- A1 pad 16: unconnected-(A1-GPIO12-Pad16) -> RPM_FAN6
- A1 pad 17: unconnected-(A1-GPIO13-Pad17) -> PWM_FAN6
- A1 pad 2: RPM_FAN1 -> unconnected-(A1-GPIO1-Pad2)
- A1 pad 4: PWM_FAN2 -> RPM_FAN1
- A1 pad 5: RPM_FAN2 -> PWM_FAN1
- A1 pad 6: PWM_FAN3 -> RPM_FAN2
- A1 pad 7: RPM_FAN3 -> PWM_FAN2
- A1 pad 9: PWM_FAN4 -> RPM_FAN3
Routing:
- net Net-(Fan6-Tacho): track 37.7 -> 41.5 mm
- net Net-(Fan3-Tacho): track 14.3 -> 10.6 mm
- net PWM_FAN3: track 25.2 -> 21.7 mm
- net Net-(Fan4-Tacho): track 19.0 -> 17.6 mm
- net PWM_FAN6: track 50.5 -> 51.8 mm
- net ADC_2: track 35.4 -> 36.5 mm
- net Net-(Fan2-Tacho): track 7.90 -> 6.95 mm
- net USB_GND: track 18.8 -> 19.7 mm
- net Net-(Fan1-Tacho): track 5.70 -> 6.55 mm
- net PWM_FAN5: track 48.5 -> 47.8 mm
- net USB_DM: track 20.1 -> 20.8 mm
- net PWM_FAN1: track 17.6 -> 18.3 mm
- net PWM_FAN2: track 19.3 -> 18.7 mm
- net ADC_1: track 31.8 -> 32.5 mm
- net USB_DP: track 20.2 -> 20.8 mm
Other:
- board text added: "VCC"
- board text added: "WayWayWay"
- board text added: "https://github.com/mietzen/RP-Pico-Fan-Controller"
- board text removed: "https://github.com/mietzen/RP2040-Fan-Controller"
- board text removed: "⊕"
- board text removed: "⊖"
