File: RP2040_Fan_Controller/RP2040_Fan_Controller.kicad_sch (KiCad schematic)
At the start: 0 parts

Commit message: PCB-Rev 0.1.0
Parts:
- added A?: RaspberryPi_Pico, Module:RaspberryPi_Pico_Common_Unspecified, symbol MCU_Module:RaspberryPi_Pico
- added Fan1, Fan2, Fan3, Fan4, Fan5, Fan6: Fan_4pin, Connector_PinSocket_2.54mm:PinSocket_1x04_P2.54mm_Horizontal, symbol Motor:Fan_4pin
- added Q10, Q11, Q12, Q7, Q8, Q9: IRLZ44N, Package_TO_SOT_THT:TO-220-3_Vertical, symbol Transistor_FET:IRLZ44N
- added R1, R2, R3: 10k, Resistor_THT:R_Axial_DIN0204_L3.6mm_D1.6mm_P5.08mm_Vertical, symbol Device:R_Small
- added R4, R5, R6, R7, R8, R9: 2.7K, Resistor_THT:R_Axial_DIN0204_L3.6mm_D1.6mm_P5.08mm_Vertical, symbol Device:R_Small
- added TH1, TH2, TH3: 10k, Connector_PinSocket_2.54mm:PinSocket_1x02_P2.54mm_Horizontal, symbol Device:Thermistor_NTC
Connections:
- new net: A?.19 (GPIO14), Q9.1 (G)
- new net: Fan3.1 (-), Q9.3 (S)
- new net: A?.20 (GPIO15), Q10.1 (G)
- new net: Fan4.1 (-), Q10.3 (S)
- new net: Fan4.3 (Tacho), R7.1
- new net: A?.12 (GPIO9), R7.2
- new net: Fan1.1 (-), Q7.3 (S)
- new net: Fan1.3 (Tacho), R4.1
- new net: A?.1 (GPIO0), Fan1.4 (PWM)
- new net: Fan5.1 (-), Q11.3 (S)
- new net: Fan5.3 (Tacho), R8.1
- new net: A?.6 (GPIO4), Fan5.4 (PWM)
- new net: A?.10 (GPIO7), R5.2
- new net: A?.11 (GPIO8), R6.2
- new net: A?.14 (GPIO10), R8.2
- new net: A?.15 (GPIO11), R9.2
- new net: A?.16 (GPIO12), Q7.1 (G)
- new net: A?.17 (GPIO13), Q8.1 (G)
- new net: A?.2 (GPIO1), Fan2.4 (PWM)
- new net: A?.21 (GPIO16), Q12.1 (G)
- new net: A?.22 (GPIO17), Q11.1 (G)
- new net: A?.31 (GPIO26_ADC0), R1.2, TH1.1
- new net: A?.32 (GPIO27_ADC1), R2.2, TH2.1
- new net: A?.33 (AGND), R1.1, R2.1, R3.1
- new net: A?.34 (GPIO28_ADC2), R3.2, TH3.1
- new net: A?.35 (ADC_VREF), TH1.2, TH2.2, TH3.2
- new net: A?.4 (GPIO2), Fan3.4 (PWM)
- new net: A?.5 (GPIO3), Fan4.4 (PWM)
- new net: A?.7 (GPIO5), Fan6.4 (PWM)
- new net: A?.9 (GPIO6), R4.2
- new net: Fan2.1 (-), Q8.3 (S)
- new net: Fan3.3 (Tacho), R6.1
- new net: Fan2.3 (Tacho), R5.1
- new net: Fan6.3 (Tacho), R9.1
- new net: Fan6.1 (-), Q12.3 (S)
- new net +12V: Fan1.2 (+), Fan2.2 (+), Fan3.2 (+), Fan4.2 (+), Fan5.2 (+), Fan6.2 (+)
- new net GND: A?.13 (GND), A?.18 (GND), A?.23 (GND), A?.28 (GND), A?.3 (GND), A?.38 (GND), A?.8 (GND), Q10.2 (D), Q11.2 (D), Q12.2 (D), Q7.2 (D), Q8.2 (D), Q9.2 (D)
Other:
- title: (none) -> RP2040 Fan Controller

Commit message: PCB-Rev 0.2.0
Parts:
- removed Q10, Q11, Q12, Q7, Q8, Q9: IRLZ44N, Package_TO_SOT_THT:TO-220-3_Vertical, symbol Transistor_FET:IRLZ44N
- added R10: 10K, Resistor_THT:R_Axial_DIN0204_L3.6mm_D1.6mm_P5.08mm_Vertical, symbol Device:R_Small
- added R11, R12, R13, R14, R15: 10k, Resistor_THT:R_Axial_DIN0204_L3.6mm_D1.6mm_P5.08mm_Vertical, symbol Device:R_Small
Connections:
- net GND: now also Fan1.1 (-), Fan2.1 (-), Fan3.1 (-), Fan4.1 (-), Fan5.1 (-), Fan6.1 (-), R10.1, R11.1, R12.1, R13.1, R14.1, R15.1
- net at A?.1 (GPIO0), Fan1.4 (PWM): now also R10.2
- net at A?.6 (GPIO4), Fan5.4 (PWM): now also R14.2
- net at A?.2 (GPIO1), Fan2.4 (PWM): now also R11.2
- net at A?.4 (GPIO2), Fan3.4 (PWM): now also R12.2
- net at A?.5 (GPIO3), Fan4.4 (PWM): now also R13.2
- net at A?.7 (GPIO5), Fan6.4 (PWM): now also R15.2

Commit message: PCB-Rev 0.2.1
Parts:
- Fan1, Fan2, Fan3, Fan4, Fan5, Fan6: footprint Connector_PinSocket_2.54mm:PinSocket_1x04_P2.54mm_Horizontal -> Connector_PinHeader_2.54mm:PinHeader_1x04_P2.54mm_Horizontal
- R1, R10, R11, R12, R13, R14, R15, R2, R3, R4, R5, R6, R7, R8, R9: footprint Resistor_THT:R_Axial_DIN0204_L3.6mm_D1.6mm_P5.08mm_Vertical -> Resistor_THT:R_Axial_DIN0204_L3.6mm_D1.6mm_P5.08mm_Horizontal
- TH1, TH2, TH3: footprint Connector_PinSocket_2.54mm:PinSocket_1x02_P2.54mm_Horizontal -> Connector_PinHeader_2.54mm:PinHeader_1x02_P2.54mm_Horizontal
- gave numbers to parts that had none: 1
Changed lines of the file:
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@@
 			)
 		)
-		(property "Footprint" "Resistor_THT:R_Axial_DIN0204_L3.6mm_D1.6mm_P5.08mm_Vertical"
+		(property "Footprint" "Resistor_THT:R_Axial_DIN0204_L3.6mm_D1.6mm_P5.08mm_Horizontal"
 			(at 87.63 38.1 0)
 			(effects
@@
 			)
 		)
-		(property "Footprint" "Resistor_THT:R_Axial_DIN0204_L3.6mm_D1.6mm_P5.08mm_Vertical"
+		(property "Footprint" "Resistor_THT:R_Axial_DIN0204_L3.6mm_D1.6mm_P5.08mm_Horizontal"
 			(at 99.06 76.2 0)
 			(effects
@@
 			)
 		)
-		(property "Footprint" "Connector_PinSocket_2.54mm:PinSocket_1x04_P2.54mm_Horizontal"
+		(property "Footprint" "Connector_PinHeader_2.54mm:PinHeader_1x04_P2.54mm_Horizontal"
 			(at 34.29 118.364 0)
 			(effects
@@
 			)
 		)
-		(property "Footprint" "Connector_PinSocket_2.54mm:PinSocket_1x04_P2.54mm_Horizontal"
+		(property "Footprint" "Connector_PinHeader_2.54mm:PinHeader_1x04_P2.54mm_Horizontal"
 			(at 69.85 159.004 0)
 			(effects
@@
 			)
 		)
-		(property "Footprint" "Resistor_THT:R_Axial_DIN0204_L3.6mm_D1.6mm_P5.08mm_Vertical"
+		(property "Footprint" "Resistor_THT:R_Axial_DIN0204_L3.6mm_D1.6mm_P5.08mm_Horizontal"
 			(at 87.63 35.56 0)
 			(effects
@@
 		(dnp no)
 		(fields_autoplaced yes)
-		(property "Reference" "A?"
+		(property "Reference" "A1"
 			(at 127.8733 102.87 0)
 			(effects
@@
 			(project ""
 				(path "/7497546a-5740-438d-96fb-d2555c11b760"
-					(reference "A?")
+					(reference "A1")
 					(unit 1)
 				)
@@
 			)
 		)
-		(property "Footprint" "Connector_PinSocket_2.54mm:PinSocket_1x02_P2.54mm_Horizontal"
+		(property "Footprint" "Connector_PinHeader_2.54mm:PinHeader_1x02_P2.54mm_Horizontal"
 			(at 176.53 69.85 0)
 			(effects
@@
 			)
 		)
-		(property "Footprint" "Resistor_THT:R_Axial_DIN0204_L3.6mm_D1.6mm_P5.08mm_Vertical"
+		(property "Footprint" "Resistor_THT:R_Axial_DIN0204_L3.6mm_D1.6mm_P5.08mm_Horizontal"
 			(at 99.06 78.74 0)
 			(effects
@@
 			)
 		)
-		(property "Footprint" "Resistor_THT:R_Axial_DIN0204_L3.6mm_D1.6mm_P5.08mm_Vertical"
+		(property "Footprint" "Resistor_THT:R_Axial_DIN0204_L3.6mm_D1.6mm_P5.08mm_Horizontal"
 			(at 87.63 30.48 0)
 			(effects
@@
 			)
 		)
-		(property "Footprint" "Resistor_THT:R_Axial_DIN0204_L3.6mm_D1.6mm_P5.08mm_Vertical"
+		(property "Footprint" "Resistor_THT:R_Axial_DIN0204_L3.6mm_D1.6mm_P5.08mm_Horizontal"
 			(at 99.06 68.58 0)
 			(effects
@@
 			)
 		)
-		(property "Footprint" "Resistor_THT:R_Axial_DIN0204_L3.6mm_D1.6mm_P5.08mm_Vertical"
+		(property "Footprint" "Resistor_THT:R_Axial_DIN0204_L3.6mm_D1.6mm_P5.08mm_Horizontal"
 			(at 99.06 73.66 0)
 			(effects
@@
 			)
 		)
-		(property "Footprint" "Connector_PinSocket_2.54mm:PinSocket_1x02_P2.54mm_Horizontal"
+		(property "Footprint" "Connector_PinHeader_2.54mm:PinHeader_1x02_P2.54mm_Horizontal"
 			(at 176.53 92.71 0)
 			(effects
@@
 			)
 		)
-		(property "Footprint" "Resistor_THT:R_Axial_DIN0204_L3.6mm_D1.6mm_P5.08mm_Vertical"
+		(property "Footprint" "Resistor_THT:R_Axial_DIN0204_L3.6mm_D1.6mm_P5.08mm_Horizontal"
 			(at 165.1 69.85 0)
 			(effects
@@
 			)
 		)
-		(property "Footprint" "Resistor_THT:R_Axial_DIN0204_L3.6mm_D1.6mm_P5.08mm_Vertical"
+		(property "Footprint" "Resistor_THT:R_Axial_DIN0204_L3.6mm_D1.6mm_P5.08mm_Horizontal"
 			(at 99.06 71.12 0)
 			(effects
@@
 			)
 		)
-		(property "Footprint" "Resistor_THT:R_Axial_DIN0204_L3.6mm_D1.6mm_P5.08mm_Vertical"
+		(property "Footprint" "Resistor_THT:R_Axial_DIN0204_L3.6mm_D1.6mm_P5.08mm_Horizontal"
 			(at 87.63 43.18 0)
 			(effects
@@
 			)
 		)
-		(property "Footprint" "Connector_PinSocket_2.54mm:PinSocket_1x04_P2.54mm_Horizontal"
+		(property "Footprint" "Connector_PinHeader_2.54mm:PinHeader_1x04_P2.54mm_Horizontal"
 			(at 43.18 128.524 0)
 			(effects
@@
 			)
 		)
-		(property "Footprint" "Resistor_THT:R_Axial_DIN0204_L3.6mm_D1.6mm_P5.08mm_Vertical"
+		(property "Footprint" "Resistor_THT:R_Axial_DIN0204_L3.6mm_D1.6mm_P5.08mm_Horizontal"
 			(at 87.63 33.02 0)
 			(effects
@@
 			)
 		)
-		(property "Footprint" "Resistor_THT:R_Axial_DIN0204_L3.6mm_D1.6mm_P5.08mm_Vertical"
+		(property "Footprint" "Resistor_THT:R_Axial_DIN0204_L3.6mm_D1.6mm_P5.08mm_Horizontal"
 			(at 99.06 81.28 0)
 			(effects
@@
 			)
 		)
-		(property "Footprint" "Resistor_THT:R_Axial_DIN0204_L3.6mm_D1.6mm_P5.08mm_Vertical"
+		(property "Footprint" "Resistor_THT:R_Axial_DIN0204_L3.6mm_D1.6mm_P5.08mm_Horizontal"
 			(at 165.1 81.28 0)
 			(effects
@@
 			)
 		)
-		(property "Footprint" "Resistor_THT:R_Axial_DIN0204_L3.6mm_D1.6mm_P5.08mm_Vertical"
+		(property "Footprint" "Resistor_THT:R_Axial_DIN0204_L3.6mm_D1.6mm_P5.08mm_Horizontal"
 			(at 87.63 40.64 0)
 			(effects
@@
 			)
 		)
-		(property "Footprint" "Connector_PinSocket_2.54mm:PinSocket_1x04_P2.54mm_Horizontal"
+		(property "Footprint" "Connector_PinHeader_2.54mm:PinHeader_1x04_P2.54mm_Horizontal"
 			(at 78.74 169.164 0)
 			(effects
@@
 			)
 		)
-		(property "Footprint" "Resistor_THT:R_Axial_DIN0204_L3.6mm_D1.6mm_P5.08mm_Vertical"
+		(property "Footprint" "Resistor_THT:R_Axial_DIN0204_L3.6mm_D1.6mm_P5.08mm_Horizontal"
 			(at 165.1 92.71 0)
 			(effects
@@
 			)
 		)
-		(property "Footprint" "Connector_PinSocket_2.54mm:PinSocket_1x04_P2.54mm_Horizontal"
+		(property "Footprint" "Connector_PinHeader_2.54mm:PinHeader_1x04_P2.54mm_Horizontal"
 			(at 60.96 148.844 0)
 			(effects
@@
 			)
 		)
-		(property "Footprint" "Connector_PinSocket_2.54mm:PinSocket_1x04_P2.54mm_Horizontal"
+		(property "Footprint" "Connector_PinHeader_2.54mm:PinHeader_1x04_P2.54mm_Horizontal"
 			(at 52.07 138.684 0)
 			(effects
@@
 			)
 		)
-		(property "Footprint" "Connector_PinSocket_2.54mm:PinSocket_1x02_P2.54mm_Horizontal"
+		(property "Footprint" "Connector_PinHeader_2.54mm:PinHeader_1x02_P2.54mm_Horizontal"
 			(at 176.53 81.28 0)
 			(effects

Commit message: PCB-Rev 0.3.0
Parts:
- removed R10: 10K, Resistor_THT:R_Axial_DIN0204_L3.6mm_D1.6mm_P5.08mm_Horizontal, symbol Device:R_Small
- removed R11, R12, R13, R14, R15: 10k, Resistor_THT:R_Axial_DIN0204_L3.6mm_D1.6mm_P5.08mm_Horizontal, symbol Device:R_Small

Commit message: PCB-Rev 0.4.0
Parts:
- removed A1: RaspberryPi_Pico, Module:RaspberryPi_Pico_Common_Unspecified, symbol MCU_Module:RaspberryPi_Pico
- added A1: RaspberryPi_Pico, Module:RaspberryPi_Pico_SMD, symbol MCU_Module:RaspberryPi_Pico_Extensive
- added J1: USB_HEADER, Connector_PinHeader_2.54mm:PinHeader_1x05_P2.54mm_Horizontal, symbol Connector:USB_B
Connections:
- net GND: now also A1.13 (GND), A1.18 (GND), A1.23 (GND), A1.28 (GND), A1.3 (GND), A1.38 (GND), A1.8 (GND), A1.D2 (GND), J1.5 (Shield)
- net RPM_FAN4: now reaches R7.2
- net RPM_FAN4: now also A1.10 (GPIO7)
- net PWM_FAN1: now reaches Fan1.4 (PWM)
- net PWM_FAN1: now also A1.1 (GPIO0)
- net PWM_FAN5: now reaches Fan5.4 (PWM)
- net PWM_FAN5: now also A1.11 (GPIO8)
- net RPM_FAN2: now reaches R5.2
- net RPM_FAN2: now also A1.5 (GPIO3)
- net RPM_FAN3: now reaches R6.2
- net RPM_FAN3: now also A1.7 (GPIO5)
- net RPM_FAN5: now reaches R8.2
- net RPM_FAN5: now also A1.12 (GPIO9)
- net RPM_FAN6: now reaches R9.2
- net RPM_FAN6: now also A1.15 (GPIO11)
- net PWM_FAN2: now reaches Fan2.4 (PWM)
- net PWM_FAN2: now also A1.4 (GPIO2)
- net ADC_0: now reaches R1.2, TH1.1
- net ADC_0: now also A1.31 (GPIO26_ADC0)
- net ADC_1: now reaches R2.2, TH2.1
- net ADC_1: now also A1.32 (GPIO27_ADC1)
- net ADC_GND: now reaches R1.1, R2.1, R3.1
- net ADC_GND: now also A1.33 (AGND)
- net ADC_2: now reaches R3.2, TH3.1
- net ADC_2: now also A1.34 (GPIO28_ADC2)
- net ADC_VREF: now reaches TH1.2, TH2.2, TH3.2
- net ADC_VREF: now also A1.35 (ADC_VREF)
- net PWM_FAN3: now reaches Fan3.4 (PWM)
- net PWM_FAN3: now also A1.6 (GPIO4)
- net PWM_FAN4: now reaches Fan4.4 (PWM)
- net PWM_FAN4: now also A1.9 (GPIO6)
- net PWM_FAN6: now reaches Fan6.4 (PWM)
- net PWM_FAN6: now also A1.14 (GPIO10)
- net RPM_FAN1: now reaches R4.2
- net RPM_FAN1: now also A1.2 (GPIO1)
- new net USB_DM: A1.TP2 (USB_DM), J1.2 (D-)
- new net USB_DP: A1.TP3 (USB_DP), J1.3 (D+)
- new net USB_GND: A1.TP1 (USB_GND), J1.4 (GND)
- new net VBUS: A1.40 (VBUS), J1.1 (VBUS)
Other:
- moved on the sheet: Fan1, Fan2, Fan3, Fan4, Fan5, Fan6, R1, R2, R3, R4, R5, R6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

Commit message: PCB-Rev 1.0.0
Parts:
- R1: renamed from R4; footprint Resistor_THT:R_Axial_DIN0204_L3.6mm_D1.6mm_P5.08mm_Horizontal -> Resistor_THT:R_Axial_DIN0204_L3.6mm_D1.6mm_P7.62mm_Horizontal
- R2: renamed from R5; footprint Resistor_THT:R_Axial_DIN0204_L3.6mm_D1.6mm_P5.08mm_Horizontal -> Resistor_THT:R_Axial_DIN0204_L3.6mm_D1.6mm_P7.62mm_Horizontal
- R3: renamed from R6; footprint Resistor_THT:R_Axial_DIN0204_L3.6mm_D1.6mm_P5.08mm_Horizontal -> Resistor_THT:R_Axial_DIN0204_L3.6mm_D1.6mm_P7.62mm_Horizontal
- R4: renamed from R7; footprint Resistor_THT:R_Axial_DIN0204_L3.6mm_D1.6mm_P5.08mm_Horizontal -> Resistor_THT:R_Axial_DIN0204_L3.6mm_D1.6mm_P7.62mm_Horizontal
- R5: renamed from R8; footprint Resistor_THT:R_Axial_DIN0204_L3.6mm_D1.6mm_P5.08mm_Horizontal -> Resistor_THT:R_Axial_DIN0204_L3.6mm_D1.6mm_P7.62mm_Horizontal
- R6: renamed from R9; footprint Resistor_THT:R_Axial_DIN0204_L3.6mm_D1.6mm_P5.08mm_Horizontal -> Resistor_THT:R_Axial_DIN0204_L3.6mm_D1.6mm_P7.62mm_Horizontal
- R7: renamed from R1; footprint Resistor_THT:R_Axial_DIN0204_L3.6mm_D1.6mm_P5.08mm_Horizontal -> Resistor_THT:R_Axial_DIN0204_L3.6mm_D1.6mm_P7.62mm_Horizontal
- R8: renamed from R2; footprint Resistor_THT:R_Axial_DIN0204_L3.6mm_D1.6mm_P5.08mm_Horizontal -> Resistor_THT:R_Axial_DIN0204_L3.6mm_D1.6mm_P7.62mm_Horizontal
- R9: renamed from R3; footprint Resistor_THT:R_Axial_DIN0204_L3.6mm_D1.6mm_P5.08mm_Horizontal -> Resistor_THT:R_Axial_DIN0204_L3.6mm_D1.6mm_P7.62mm_Horizontal
Connections:
- net PWM_FAN1: now also A1.5 (GPIO3); no longer A1.1 (GPIO0)
- net PWM_FAN2: now also A1.7 (GPIO5); no longer A1.4 (GPIO2)
- net PWM_FAN3: now also A1.10 (GPIO7); no longer A1.6 (GPIO4)
- net PWM_FAN4: now also A1.12 (GPIO9); no longer A1.9 (GPIO6)
- net PWM_FAN5: now also A1.15 (GPIO11); no longer A1.11 (GPIO8)
- net PWM_FAN6: now also A1.17 (GPIO13); no longer A1.14 (GPIO10)
- net RPM_FAN1: now also A1.4 (GPIO2); no longer A1.2 (GPIO1)
- net RPM_FAN2: now also A1.6 (GPIO4); no longer A1.5 (GPIO3)
- net RPM_FAN3: now also A1.9 (GPIO6); no longer A1.7 (GPIO5)
- net RPM_FAN4: now also A1.11 (GPIO8); no longer A1.10 (GPIO7)
- net RPM_FAN5: now also A1.14 (GPIO10); no longer A1.12 (GPIO9)
- net RPM_FAN6: now also A1.16 (GPIO12); no longer A1.15 (GPIO11)
